File: PCB/Button/ju_button.kicad_pcb (KiCad board)
At the start: 2 copper layers, 103.2 x 107.2 mm, 17 parts, among them J1 Conn_01x05

Commit message: PCBs of v1.1
Parts:
- moved J1 2.00 mm to (136.9, 63.9)
Routing:
- net GND: track 558.7 -> 579.6 mm
- net Net-(B1-A): track 139.5 -> 147.7 mm, vias 2 -> 3
- net Net-(C1-B): track 194.9 -> 202.8 mm
- net Net-(D1-A): track 193.8 -> 199.4 mm
Other:
- board size 103.2 x 107.2 mm -> 103.2 x 105.2 mm
- board text added: "Button v1.1"
- board text removed: "Button v1.0"

Commit message: Button PCB v1.2 files (missing from previous commit)
Parts:
- moved A1 1.50 mm to (97.4, 65.7)
- moved A2 1.50 mm to (92.5, 107.6)
- moved A3 1.50 mm to (134.4, 112.5)
- moved A4 1.50 mm to (139.3, 70.6)
- moved B1 1.50 mm to (147.4, 65.7)
- moved B2 1.50 mm to (142.5, 107.6)
- moved B3 1.50 mm to (184.4, 112.5)
- moved B4 1.50 mm to (189.3, 70.6)
- moved C1 1.50 mm to (97.4, 115.7)
- moved C2 1.50 mm to (92.5, 157.6)
- moved C3 1.50 mm to (134.4, 162.5)
- moved C4 1.50 mm to (139.3, 120.6)
- moved D1 1.50 mm to (147.4, 115.7)
- moved D2 1.50 mm to (142.5, 157.6)
- moved D3 1.50 mm to (184.4, 162.5)
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Routing:
- net Net-(B1-A): track 147.7 -> 144.9 mm
- net Net-(C1-B): track 202.8 -> 200.6 mm
- net Net-(D1-A): track 199.4 -> 201.3 mm
- net GND: track 579.6 -> 580.2 mm
- net Net-(A1-B): track 140.8 -> 140.2 mm
Other:
- outline, holes or cut-outs redrawn
- board text added: "Button v1.2"
- board text removed: "Button v1.1"
- board text removed: "JLCJLCJLCJLC"
