File: PCB/IO/ju_io.kicad_sch (KiCad schematic)
At the start: 17 parts, among them J1 Conn_01x05, J2 Conn_01x05, J3 Conn_01x05, J4 Conn_01x05, J5 Conn_01x03, J6 Conn_01x03, U1 PiPico_No_SWD

Commit message: PCBs of v1.1
Parts:
- removed J6: Conn_01x03, ju_io:SH1.0_3P, symbol Connector_Generic:Conn_01x03
- added D1, D2, D3, D4: WS2812B_Unified, ju_io:WS2812B-2835, symbol musec_pico:WS2812B_Unified
- U1: footprint ju_io:RPi_Pico_SMD_Pins_No_SWD -> ju_io:RPi_Pico_SMD_Pins_No_SWD_No_Text
Connections:
- net +5V: now also D1.V (VDD), D2.V (VDD), D3.V (VDD), D4.V (VDD)
- net GND: now also D1.G (VSS), D2.G (VSS), D3.G (VSS), D4.G (VSS)
- net at U1.21 (GPIO16): no longer R4.1
- net at U1.34 (GPIO28_ADC2): now also R4.1
- net at R4.2: now also J5.2 (Pin_2)
- net at R3.2: now also D1.I (In); no longer J5.2 (Pin_2)
- new net: D3.O (Out), D4.I (In)
- new net: D1.O (Out), D2.I (In)
- new net: D2.O (Out), D3.I (In)
- no-connect marks 10 -> 11
Other:
- moved on the sheet: C1, R3, R4

Commit message: PCB optimization button v1.2, io v1.21
Parts:
- B1, B2, B3, B4: footprint ju_io:SKSTAAE010 -> ju_io:EVQP1K05M
Changed lines of the file:
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@@
 			)
 		)
-		(property "Footprint" "ju_io:SKSTAAE010"
+		(property "Footprint" "ju_io:EVQP1K05M"
 			(at 240.665 166.37 0)
 			(effects
@@
 			)
 		)
-		(property "Footprint" "ju_io:SKSTAAE010"
+		(property "Footprint" "ju_io:EVQP1K05M"
 			(at 240.665 172.72 0)
 			(effects
@@
 			)
 		)
-		(property "Footprint" "ju_io:SKSTAAE010"
+		(property "Footprint" "ju_io:EVQP1K05M"
 			(at 240.665 179.07 0)
 			(effects
@@
 			)
 		)
-		(property "Footprint" "ju_io:SKSTAAE010"
+		(property "Footprint" "ju_io:EVQP1K05M"
 			(at 240.665 160.02 0)
 			(effects

Commit message: Ju Pico IO PCB v1.22
Parts:
- removed R3, R4: 10, Resistor_SMD:R_0603_1608Metric_Pad0.98x0.95mm_HandSolder, symbol Device:R_Small
Connections:
- net at J5.2 (Pin_2): now also U1.34 (GPIO28_ADC2)
- net at U1.22 (GPIO17): now also D1.I (In)
Changed lines of the file:
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@@
 (kicad_sch
-	(version 20231120)
+	(version 20250114)
 	(generator "eeschema")
-	(generator_version "8.0")
+	(generator_version "9.0")
 	(paper "A3")
 	(junction
@@
 	(wire
 		(pts
-			(xy 218.44 184.15) (xy 274.32 184.15)
+			(xy 218.44 184.15) (xy 293.37 184.15)
 		)
 		(stroke
@@
 	(wire
 		(pts
-			(xy 218.44 153.67) (xy 252.73 153.67)
+			(xy 218.44 153.67) (xy 266.065 153.67)
 		)
 		(stroke
@@
 	(wire
 		(pts
-			(xy 257.81 153.67) (xy 266.065 153.67)
-		)
-		(stroke
-			(width 0)
-			(type default)
-		)
-	)
-	(wire
-		(pts
 			(xy 325.12 196.215) (xy 325.12 191.77)
 		)
@@
 	(wire
 		(pts
-			(xy 279.4 184.15) (xy 293.37 184.15)
-		)
-		(stroke
-			(width 0)
-			(type default)
-		)
-	)
-	(wire
-		(pts
 			(xy 223.52 66.675) (xy 223.52 138.43)
 		)
@@
 	)
 	(symbol
-		(lib_id "Device:R_Small")
-		(at 255.27 153.67 90)
-		(unit 1)
-		(exclude_from_sim no)
-		(in_bom yes)
-		(on_board yes)
-		(dnp no)
-		(property "Reference" "R4"
-			(at 256.54 151.765 90)
-			(effects
-				(font
-					(size 1.27 1.27)
-				)
-				(justify left)
-			)
-		)
-		(property "Value" "10"
-			(at 256.54 155.575 90)
-			(effects
-				(font
-					(size 1.27 1.27)
-				)
-				(justify left)
-			)
-		)
-		(property "Footprint" "Resistor_SMD:R_0603_1608Metric_Pad0.98x0.95mm_HandSolder"
-			(at 255.27 153.67 0)
-			(effects
-				(font
-					(size 1.27 1.27)
-				)
-				(hide yes)
-			)
-		)
-		(property "Datasheet" "~"
-			(at 255.27 153.67 0)
-			(effects
-				(font
-					(size 1.27 1.27)
-				)
-				(hide yes)
-			)
-		)
-		(property "Description" ""
-			(at 255.27 153.67 0)
-			(effects
-				(font
-					(size 1.27 1.27)
-				)
-				(hide yes)
-			)
-		)
-		(property "LCSC" "C23186"
-			(at 255.27 153.67 0)
-			(effects
-				(font
-					(size 1.27 1.27)
-				)
-				(hide yes)
-			)
-		)
-		(pin "1"
-		)
-		(pin "2"
-		)
-		(instances
-			(project "ju_io"
-				(path "/2e3f5573-c264-4a8b-a2f0-0e6473d39aad"
-					(reference "R4")
-					(unit 1)
-				)
-			)
-		)
-	)
-	(symbol
 		(lib_id "Switch:SW_SPST")
 		(at 240.665 172.72 0)
@@
 	)
 	(symbol
-		(lib_id "Device:R_Small")
-		(at 276.86 184.15 90)
-		(unit 1)
-		(exclude_from_sim no)
-		(in_bom yes)
-		(on_board yes)
-		(dnp no)
-		(property "Reference" "R3"
-			(at 278.13 182.245 90)
-			(effects
-				(font
-					(size 1.27 1.27)
-				)
-				(justify left)
-			)
-		)
-		(property "Value" "10"
-			(at 278.13 186.055 90)
-			(effects
-				(font
-					(size 1.27 1.27)
-				)
-				(justify left)
-			)
-		)
-		(property "Footprint" "Resistor_SMD:R_0603_1608Metric_Pad0.98x0.95mm_HandSolder"
-			(at 276.86 184.15 0)
-			(effects
-				(font
-					(size 1.27 1.27)
-				)
-				(hide yes)
-			)
-		)
-		(property "Datasheet" "~"
-			(at 276.86 184.15 0)
-			(effects
-				(font
-					(size 1.27 1.27)
-				)
-				(hide yes)
-			)
-		)
-		(property "Description" ""
-			(at 276.86 184.15 0)
-			(effects
-				(font
-					(size 1.27 1.27)
-				)
-				(hide yes)
-			)
-		)
-		(property "LCSC" "C23186"
-			(at 276.86 184.15 0)
-			(effects
-				(font
-					(size 1.27 1.27)
-				)
-				(hide yes)
-			)
-		)
-		(pin "1"
-		)
-		(pin "2"
-		)
-		(instances
-			(project "ju_io"
-				(path "/2e3f5573-c264-4a8b-a2f0-0e6473d39aad"
-					(reference "R3")
-					(unit 1)
-				)
-			)
-		)
-	)
-	(symbol
 		(lib_id "Switch:SW_SPST")
 		(at 240.665 179.07 0)
@@
 		)
 	)
+	(embedded_fonts no)
 )
